File: pcb/hackpad-full-keyboard.kicad_sch (KiCad schematic)
At the start: 277 parts, among them J0 SW_Push_45deg, J2 Conn_01x04_Pin, K0 SW_Push_45deg, M0 SW_Push_45deg, P0 SW_Push_45deg, Q0 SW_Push_45deg, T0 SW_Push_45deg, U0 SW_Push_45deg, U1 Raspberry_Pi_Pico, X0 SW_Push_45deg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

Commit message: Adjust size of escape key
Parts:
- ESC0: footprint Button_Switch_Keyboard:SW_Cherry_MX_2.00u_PCB -> Button_Switch_Keyboard:SW_Cherry_MX_1.00u_PCB
Changed lines of the file:
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@@
 			)
 		)
-		(property "Footprint" "Button_Switch_Keyboard:SW_Cherry_MX_2.00u_PCB"
+		(property "Footprint" "Button_Switch_Keyboard:SW_Cherry_MX_1.00u_PCB"
 			(at 24.13 35.56 0)
 			(effects
